Commit message: Added joint control for model

File: wagon_description/urdf/wagon.urdf_gazebo.xacro (robot description, xacro)
@@ -1,16 +1,51 @@
 <?xml version="1.0" ?>
-<robot name="wagon" xmlns:xacro="http://ros.org/wiki/xacro">
-  <xacro:include filename="$(find wagon_description)/urdf/common_properties.xacro"/>
-  <xacro:property name="height" value="0.294" />
-  <xacro:property name="hydrolic_offset" value="0.085" />
+<!-- =================================================================================== -->
+<!-- |    This document was autogenerated by xacro from wagon.xacro                    | -->
+<!-- |    EDITING THIS FILE BY HAND IS NOT RECOMMENDED                                 | -->
+<!-- =================================================================================== -->
+<robot name="wagon">
+  <!-- Init colour -->
+  <material name="black">
+    <color rgba="0.0 0.0 0.0 1.0"/>
+  </material>
+  <material name="dark">
+    <color rgba="0.3 0.3 0.3 1.0"/>
+  </material>
+  <material name="light_black">
+    <color rgba="0.4 0.4 0.4 1.0"/>
+  </material>
+  <material name="blue">
+    <color rgba="0.0 0.0 0.8 1.0"/>
+  </material>
+  <material name="green">
+    <color rgba="0.0 0.8 0.0 1.0"/>
+  </material>
+  <material name="grey">
+    <color rgba="0.5 0.5 0.5 1.0"/>
+  </material>
+  <material name="orange">
+    <color rgba="1.0 0.4235294117647059 0.0392156862745098 1.0"/>
+  </material>
+  <material name="brown">
+    <color rgba="0.8705882352941177 0.8117647058823529 0.7647058823529411 1.0"/>
+  </material>
+  <material name="red">
+    <color rgba="0.8 0.0 0.0 1.0"/>
+  </material>
+  <material name="white">
+    <color rgba="1.0 1.0 1.0 1.0"/>
+  </material>
+  <material name="acrylic">
+    <color rgba="0.9 0.9 1.0 0.6"/>
+  </material>
   <link name="base_footprint"/>
   <joint name="base_joint" type="fixed">
     <parent link="base_footprint"/>
     <child link="base_link"/>
-    <origin xyz="0.6948 0 0" rpy="0 0 0"/>
+    <origin rpy="0 0 0" xyz="0.6948 0 0"/>
   </joint>
   <link name="base_link">
     <visual>
-      <origin xyz="0 0 0" rpy="0 0 1.57"/>
+      <origin rpy="0 0 1.57" xyz="0 0 0"/>
       <geometry>
         <mesh filename="$(find wagon_description)/meshes/bases/Simplified_Front_Centered.stl" scale="0.001 0.001 0.001"/>
@@ -19,5 +54,5 @@
     </visual>
     <collision>
-      <origin xyz="-${0.6948-(1.055/2)+0.02} 0 0" rpy="0 0 0"/>
+      <origin rpy="0 0 0" xyz="-0.1873 0 0"/>
       <geometry>
         <box size="1.055 0.620 0.260"/>
@@ -25,9 +60,7 @@
     </collision>
     <inertial>
-      <origin xyz="-0.142 0 0" rpy="0 ${pi/2} 0" />
-      <mass value="135.5" />
-      <inertia ixx="6.189"
-               ixy="0" iyy="17.997"
-               ixz="-0.009" iyz="0" izz="21.229" />
+      <origin rpy="0 1.5707963267948966 0" xyz="-0.142 0 0"/>
+      <mass value="135.5"/>
+      <inertia ixx="6.189" ixy="0" ixz="-0.009" iyy="17.997" iyz="0" izz="21.229"/>
     </inertial>
   </link>
@@ -35,5 +68,5 @@
     <axis xyz="0 0 1"/>
     <limit effort="1000.0" lower="-0.550" upper="0.550" velocity="0.5"/>
-    <origin rpy="0 0 0" xyz="${-0.6948-hydrolic_offset} 0.0 0"/>
+    <origin rpy="0 0 0" xyz="-0.7797999999999999 0.0 0"/>
     <parent link="base_link"/>
     <child link="hydrolic_link"/>
@@ -44,28 +77,26 @@
     <parent link="hydrolic_link"/>
     <child link="rear_link"/>
-    <origin xyz="${-0.8716+hydrolic_offset} 0 0" rpy="0 0 0"/>
+    <origin rpy="0 0 0" xyz="-0.7866000000000001 0 0"/>
   </joint>
   <link name="rear_link">
     <visual>
-        <origin xyz="0 0 0" rpy="0 0 1.57"/>
-        <geometry>
+      <origin rpy="0 0 1.57" xyz="0 0 0"/>
+      <geometry>
         <mesh filename="$(find wagon_description)/meshes/bases/Simplified_Back_Centered.stl" scale="0.001 0.001 0.001"/>
-        </geometry>
-        <material name="white"/>
-    </visual>
-<!-- ${-0.8716+hydrolic_offset-(1.180/2)+0.02} -->
-<!-- ${(1.180/2) + 0.8716+hydrolic_offset+0.02-1.180} -->
-    <collision>
-        <origin xyz="${0.09} 0 0" rpy="0 0 0"/>
-        <geometry>
-        <box size="${1.02} 0.620 0.260"/>
-        </geometry>
-    </collision>
-    <inertial>
-        <origin xyz="${0.142} 0 0" rpy="0 0 0" />
-        <mass value="140.5" />
-      <inertia ixx="6.189"
-               ixy="0" iyy="17.997"
-               ixz="-0.009" iyz="0" izz="21.229" />
+      </geometry>
+      <material name="white"/>
+    </visual>
+    <!-- ${-0.8716+hydrolic_offset-(1.180/2)+0.02} -->
+    <!-- ${(1.180/2) + 0.8716+hydrolic_offset+0.02-1.180} -->
+    <collision>
+      <origin rpy="0 0 0" xyz="0.09 0 0"/>
+      <geometry>
+        <box size="1.02 0.620 0.260"/>
+      </geometry>
+    </collision>
+    <inertial>
+      <origin rpy="0 0 0" xyz="0.142 0 0"/>
+      <mass value="140.5"/>
+      <inertia ixx="6.189" ixy="0" ixz="-0.009" iyy="17.997" iyz="0" izz="21.229"/>
     </inertial>
   </link>
@@ -73,22 +104,22 @@
     <parent link="base_link"/>
     <child link="wheel_front_right_link"/>
-    <origin xyz="0 -0.4815 0" rpy="0 0 0"/>
+    <origin rpy="0 0 0" xyz="0 -0.4815 0"/>
     <axis xyz="0 1 0"/>
   </joint>
   <link name="wheel_front_right_link">
     <visual>
-      <origin xyz="0 0 0" rpy="1.57 0 0"/>
-      <geometry>
-        <mesh filename="$(find wagon_description)/meshes/wheels/Wheel.stl" scale="0.001 0.001 0.001"/>
-      <!--
-      <origin xyz="0 0 0" rpy="0 0 0"/>
-      <geometry>
-        <cylinder length="0.07" radius="0.12"/>
-        -->
-      </geometry>
-      <material name="black"/>
-    </visual>
-    <collision>
-      <origin xyz="0 0 0" rpy="1.57 0 0"/>
+      <origin rpy="1.57 0 0" xyz="0 0 0"/>
+      <geometry>
+        <mesh filename="$(find wagon_description)/meshes/wheels/Wheel.stl" scale="0.001 0.001 0.001"/>
+        <!--
+      <origin xyz="0 0 0" rpy="0 0 0"/>
+      <geometry>
+        <cylinder length="0.07" radius="0.12"/>
+        -->
+      </geometry>
+      <material name="black"/>
+    </visual>
+    <collision>
+      <origin rpy="1.57 0 0" xyz="0 0 0"/>
       <geometry>
         <cylinder length="0.215" radius="0.292"/>
@@ -96,32 +127,30 @@
     </collision>
     <inertial>
-      <origin xyz="0 0 0" rpy="1.57 0 0" />
-      <mass value="40.5" />
-      <inertia ixx="1.05"
-               ixy="1.0783e-10" iyy="1.83"
-               ixz="-0.023" iyz="-0.898e-11" izz="1.05" />
-    </inertial>
-  </link>
-    <joint name="wheel_front_left_joint" type="continuous">
+      <origin rpy="1.57 0 0" xyz="0 0 0"/>
+      <mass value="40.5"/>
+      <inertia ixx="1.05" ixy="1.0783e-10" ixz="-0.023" iyy="1.83" iyz="-0.898e-11" izz="1.05"/>
+    </inertial>
+  </link>
+  <joint name="wheel_front_left_joint" type="continuous">
     <parent link="base_link"/>
     <child link="wheel_front_left_link"/>
-    <origin xyz="0 0.4815 0" rpy="0 0 0"/>
+    <origin rpy="0 0 0" xyz="0 0.4815 0"/>
     <axis xyz="0 1 0"/>
   </joint>
   <link name="wheel_front_left_link">
     <visual>
-      <origin xyz="0 0 0" rpy="1.57 0 0"/>
-      <geometry>
-        <mesh filename="$(find wagon_description)/meshes/wheels/Wheel.stl" scale="0.001 0.001 0.001"/>
-      <!--
-      <origin xyz="0 0 0" rpy="0 0 0"/>
-      <geometry>
-        <cylinder length="0.07" radius="0.12"/>
-        -->
-      </geometry>
-      <material name="black"/>
-    </visual>
-    <collision>
-      <origin xyz="0 0 0" rpy="1.57 0 0"/>
+      <origin rpy="1.57 0 0" xyz="0 0 0"/>
+      <geometry>
+        <mesh filename="$(find wagon_description)/meshes/wheels/Wheel.stl" scale="0.001 0.001 0.001"/>
+        <!--
+      <origin xyz="0 0 0" rpy="0 0 0"/>
+      <geometry>
+        <cylinder length="0.07" radius="0.12"/>
+        -->
+      </geometry>
+      <material name="black"/>
+    </visual>
+    <collision>
+      <origin rpy="1.57 0 0" xyz="0 0 0"/>
       <geometry>
         <cylinder length="0.215" radius="0.294"/>
@@ -129,9 +158,7 @@
     </collision>
     <inertial>
-      <origin xyz="0 0 0" rpy="1.57 0 0" />
-      <mass value="40.5" />
-      <inertia ixx="1.05"
-               ixy="1.0783e-10" iyy="1.83"
-               ixz="-0.023" iyz="-0.898e-11" izz="1.05" />
+      <origin rpy="1.57 0 0" xyz="0 0 0"/>
+      <mass value="40.5"/>
+      <inertia ixx="1.05" ixy="1.0783e-10" ixz="-0.023" iyy="1.83" iyz="-0.898e-11" izz="1.05"/>
     </inertial>
   </link>
@@ -139,22 +166,22 @@
     <parent link="rear_link"/>
     <child link="wheel_rear_right_link"/>
-    <origin xyz="0 -0.4815 0" rpy="0 0 0"/>
+    <origin rpy="0 0 0" xyz="0 -0.4815 0"/>
     <axis xyz="0 1 0"/>
   </joint>
   <link name="wheel_rear_right_link">
     <visual>
-      <origin xyz="0 0 0" rpy="1.57 0 0"/>
-      <geometry>
-        <mesh filename="$(find wagon_description)/meshes/wheels/Wheel.stl" scale="0.001 0.001 0.001"/>
-      <!--
-      <origin xyz="0 0 0" rpy="0 0 0"/>
-      <geometry>
-        <cylinder length="0.07" radius="0.12"/>
-        -->
-      </geometry>
-      <material name="black"/>
-    </visual>
-    <collision>
-      <origin xyz="0 0 0" rpy="1.57 0 0"/>
+      <origin rpy="1.57 0 0" xyz="0 0 0"/>
+      <geometry>
+        <mesh filename="$(find wagon_description)/meshes/wheels/Wheel.stl" scale="0.001 0.001 0.001"/>
+        <!--
+      <origin xyz="0 0 0" rpy="0 0 0"/>
+      <geometry>
+        <cylinder length="0.07" radius="0.12"/>
+        -->
+      </geometry>
+      <material name="black"/>
+    </visual>
+    <collision>
+      <origin rpy="1.57 0 0" xyz="0 0 0"/>
       <geometry>
         <cylinder length="0.215" radius="0.294"/>
@@ -162,32 +189,30 @@
     </collision>
     <inertial>
-      <origin xyz="0 0 0" rpy="0 0 0" />
-      <mass value="40.5" />
-      <inertia ixx="1.05"
-               ixy="1.0783e-10" iyy="1.83"
-               ixz="-0.023" iyz="-0.898e-11" izz="1.05" />
-    </inertial>
-  </link>
-    <joint name="wheel_rear_left_joint" type="continuous">
+      <origin rpy="0 0 0" xyz="0 0 0"/>
+      <mass value="40.5"/>
+      <inertia ixx="1.05" ixy="1.0783e-10" ixz="-0.023" iyy="1.83" iyz="-0.898e-11" izz="1.05"/>
+    </inertial>
+  </link>
+  <joint name="wheel_rear_left_joint" type="continuous">
     <parent link="rear_link"/>
     <child link="wheel_rear_left_link"/>
-    <origin xyz="0 0.4815 0" rpy="0 0 0"/>
+    <origin rpy="0 0 0" xyz="0 0.4815 0"/>
     <axis xyz="0 1 0"/>
   </joint>
   <link name="wheel_rear_left_link">
     <visual>
-      <origin xyz="0 0 0" rpy="1.57 0 0"/>
-      <geometry>
-        <mesh filename="$(find wagon_description)/meshes/wheels/Wheel.stl" scale="0.001 0.001 0.001"/>
-      <!--
-      <origin xyz="0 0 0" rpy="0 0 0"/>
-      <geometry>
-        <cylinder length="0.07" radius="0.12"/>
-        -->
-      </geometry>
-      <material name="black"/>
-    </visual>
-    <collision>
-      <origin xyz="0 0 0" rpy="1.57 0 0"/>
+      <origin rpy="1.57 0 0" xyz="0 0 0"/>
+      <geometry>
+        <mesh filename="$(find wagon_description)/meshes/wheels/Wheel.stl" scale="0.001 0.001 0.001"/>
+        <!--
+      <origin xyz="0 0 0" rpy="0 0 0"/>
+      <geometry>
+        <cylinder length="0.07" radius="0.12"/>
+        -->
+      </geometry>
+      <material name="black"/>
+    </visual>
+    <collision>
+      <origin rpy="1.57 0 0" xyz="0 0 0"/>
       <geometry>
         <cylinder length="0.215" radius="0.294"/>
@@ -195,9 +220,7 @@
     </collision>
     <inertial>
-      <origin xyz="0 0 0" rpy="1.57 0 0" />
-      <mass value="40.5" />
-      <inertia ixx="1.05"
-               ixy="1.0783e-10" iyy="1.83"
-               ixz="-0.023" iyz="-0.898e-11" izz="1.05" />
+      <origin rpy="1.57 0 0" xyz="0 0 0"/>
+      <mass value="40.5"/>
+      <inertia ixx="1.05" ixy="1.0783e-10" ixz="-0.023" iyy="1.83" iyz="-0.898e-11" izz="1.05"/>
     </inertial>
   </link>
