Commit message: cleaned up, made gazebo wagon local

File: wagon_description/urdf/wagon_gazebo.urdf (robot description, URDF)
Before this commit: robot wagon, 8 links, 7 joints
Links:
- link base_link: geometry collision box size=1.055 0.620 0.260; visual mesh filename=meshes/bases/Simplified_Front_Centered.stl scale=0.001 0.001 0.001
- link rear_link: geometry collision box size=1.02 0.620 0.260; visual mesh filename=meshes/bases/Simplified_Back_Centered.stl scale=0.001 0.001 0.001
- link wheel_front_left_link: geometry collision cylinder length=0.215 radius=0.294; visual mesh filename=meshes/wheels/Wheel.stl scale=0.001 0.001 0.001
- link wheel_front_right_link: geometry collision cylinder length=0.215 radius=0.292; visual mesh filename=meshes/wheels/Wheel.stl scale=0.001 0.001 0.001
- link wheel_rear_left_link: geometry collision cylinder length=0.215 radius=0.294; visual mesh filename=meshes/wheels/Wheel.stl scale=0.001 0.001 0.001
- link wheel_rear_right_link: geometry collision cylinder length=0.215 radius=0.294; visual mesh filename=meshes/wheels/Wheel.stl scale=0.001 0.001 0.001
