Commit message: added inertia and mass estimates

File: wagon_description/urdf/wagon.urdf (robot description, URDF)
Before this commit: robot wagon, 8 links, 7 joints
Links:
- link base_link: mass 7.5 -> 135.5; geometry collision box size=1.055 0.620 0.260; visual mesh filename=package://wagon_description/meshes/bases/Simplified_Front_C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 scale=0.001 0.001 0.001
- link rear_link: mass 7.5 -> 140.5; geometry collision box size=1.02 0.620 0.260; visual mesh filename=package://wagon_description/meshes/bases/Simplified_Back_Ce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 scale=0.001 0.001 0.001
- link wheel_front_left_link: mass 1.525 -> 40.5; geometry collision cylinder length=0.215 radius=0.294; visual mesh filename=package://wagon_description/meshes/wheels/Wheel.stl scale=0.001 0.001 0.001
- link wheel_front_right_link: mass 1.525 -> 40.5; geometry collision cylinder length=0.215 radius=0.292; visual mesh filename=package://wagon_description/meshes/wheels/Wheel.stl scale=0.001 0.001 0.001
- link wheel_rear_left_link: mass 1.525 -> 40.5; geometry collision cylinder length=0.215 radius=0.294; visual mesh filename=package://wagon_description/meshes/wheels/Wheel.stl scale=0.001 0.001 0.001
- link wheel_rear_right_link: mass 1.525 -> 40.5; geometry collision cylinder length=0.215 radius=0.294; visual mesh filename=package://wagon_description/meshes/wheels/Wheel.stl scale=0.001 0.001 0.001

File: wagon_description/urdf/wagon.xacro (robot description, xacro)
@@ -25,9 +25,9 @@
     </collision>
     <inertial>
-      <origin xyz="-0.142 0 0" rpy="0 0 0" />
-      <mass value="7.5" />
-      <inertia ixx="4.806e-2"
-               ixy="0.0" iyy="1.193e-1"
-               ixz="0.0" iyz="0.0" izz="1.493e-1" />
+      <origin xyz="-0.142 0 0" rpy="0 ${pi/2} 0" />
+      <mass value="135.5" />
+      <inertia ixx="6.189"
+               ixy="0" iyy="17.997"
+               ixz="-0.009" iyz="0" izz="21.229" />
     </inertial>
   </link>
@@ -63,9 +63,9 @@
     </collision>
     <inertial>
-        <origin xyz="-0.142 0 0" rpy="0 0 0" />
-        <mass value="7.5" />
-        <inertia ixx="4.806e-2"
-                ixy="0.0" iyy="1.193e-1"
-                ixz="0.0" iyz="0.0" izz="1.493e-1" />
+        <origin xyz="${0.142} 0 0" rpy="0 0 0" />
+        <mass value="140.5" />
+      <inertia ixx="6.189"
+               ixy="0" iyy="17.997"
+               ixz="-0.009" iyz="0" izz="21.229" />
     </inertial>
   </link>
@@ -97,8 +97,8 @@
     <inertial>
       <origin xyz="0 0 0" rpy="1.57 0 0" />
-      <mass value="1.525" />
-      <inertia ixx="6.723e-3"
-               ixy="0.0" iyy="6.723e-3"
-               ixz="0.0" iyz="0.0" izz="1.220e-2" />
+      <mass value="40.5" />
+      <inertia ixx="1.05"
+               ixy="1.0783e-10" iyy="1.83"
+               ixz="-0.023" iyz="-0.898e-11" izz="1.05" />
     </inertial>
   </link>
@@ -130,11 +130,11 @@
     <inertial>
       <origin xyz="0 0 0" rpy="1.57 0 0" />
-      <mass value="1.525" />
-      <inertia ixx="6.723e-3"
-               ixy="0.0" iyy="6.723e-3"
-               ixz="0.0" iyz="0.0" izz="1.220e-2" />
-    </inertial>
-  </link>
-    <joint name="wheel_rear_right_joint" type="continuous">
+      <mass value="40.5" />
+      <inertia ixx="1.05"
+               ixy="1.0783e-10" iyy="1.83"
+               ixz="-0.023" iyz="-0.898e-11" izz="1.05" />
+    </inertial>
+  </link>
+  <joint name="wheel_rear_right_joint" type="continuous">
     <parent link="rear_link"/>
     <child link="wheel_rear_right_link"/>
@@ -162,9 +162,9 @@
     </collision>
     <inertial>
-      <origin xyz="0 0 0" rpy="1.57 0 0" />
-      <mass value="1.525" />
-      <inertia ixx="6.723e-3"
-               ixy="0.0" iyy="6.723e-3"
-               ixz="0.0" iyz="0.0" izz="1.220e-2" />
+      <origin xyz="0 0 0" rpy="0 0 0" />
+      <mass value="40.5" />
+      <inertia ixx="1.05"
+               ixy="1.0783e-10" iyy="1.83"
+               ixz="-0.023" iyz="-0.898e-11" izz="1.05" />
     </inertial>
   </link>
@@ -196,8 +196,8 @@
     <inertial>
       <origin xyz="0 0 0" rpy="1.57 0 0" />
-      <mass value="1.525" />
-      <inertia ixx="6.723e-3"
-               ixy="0.0" iyy="6.723e-3"
-               ixz="0.0" iyz="0.0" izz="1.220e-2" />
+      <mass value="40.5" />
+      <inertia ixx="1.05"
+               ixy="1.0783e-10" iyy="1.83"
+               ixz="-0.023" iyz="-0.898e-11" izz="1.05" />
     </inertial>
   </link>

Commit message: added connection joint to urdf

File: wagon_description/urdf/wagon.urdf (robot description, URDF)
Before this commit: robot wagon, 9 links, 8 joints
Links:
- link rear_link: geometry collision box size=1.02 0.620 0.260; visual mesh filename=package://wagon_description/meshes/bases/Simplified_Back_Ce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 scale=0.001 0.001 0.001
Joints:
- joint connection_joint: origin xyz=${rear_link_offset + hydraulic_offset} 0 0 rpy=0 0 0 -> xyz=-0.7866000000000001 0 0 rpy=0 0 0
- joint rear_joint: origin xyz=${-0.8716+hydraulic_offset} 0 0 rpy=0 0 0 -> xyz=-0.7866000000000001 0 0 rpy=0 0 0

Commit message: Added Lidar and IMU to urdf

File: wagon_description/urdf/wagon.urdf (robot description, URDF)
Before this commit: robot wagon, 9 links, 8 joints
Links:
- added link base_scan, mass 0.314; collision cylinder length=0.072 radius=0.079; visual mesh filename=package://wagon_description/meshes/sensors/ouster_OS1.dae scale=1 1 1
- added link imu_link
Joints:
- added joint imu_joint: type fixed, parent base_link, child imu_link, origin xyz=-0.032 0 0.068 rpy=0 0 0
- added joint scan_joint: type fixed, parent base_link, child base_scan, origin xyz=0 0 0.272 rpy=0 0 0

File: wagon_description/urdf/wagon.xacro (robot description, xacro)
@@ -209,3 +209,34 @@
     </inertial>
   </link>
+  <joint name="imu_joint" type="fixed">
+    <parent link="base_link"/>
+    <child link="imu_link"/>
+    <origin xyz="-0.032 0 0.068" rpy="0 0 0"/>
+  </joint>
+  <link name="imu_link"/>
+  <joint name="scan_joint" type="fixed">
+    <parent link="base_link"/>
+    <child link="base_scan"/>
+    <origin xyz="0 0 0.272" rpy="0 0 0"/>
+  </joint>
+  <link name="base_scan">
+    <visual>
+      <origin xyz="0 0 -0.036" rpy="${pi/2} 0 0"/>
+      <geometry>
+        <mesh filename="package://wagon_description/meshes/sensors/ouster_OS1.dae" scale="1 1 1"/>
+      </geometry>
+      <material name="dark"/>
+    </visual>
+    <collision>
+      <origin xyz="0 0 -0.036" rpy="0 0 0"/>
+      <geometry>
+        <cylinder length="0.072" radius="0.079"/>
+      </geometry>
+    </collision>
+    <inertial>
+      <mass value="0.314" />
+      <origin xyz="0 0 0" />
+      <inertia ixx="0.001" ixy="0.0" ixz="0.0" iyy="0.001" iyz="0.0" izz="0.001" />
+    </inertial>
+  </link>
 </robot>

Commit message: lidar_3d, joint state, simple gps, wheel vel WIP

File: wagon_description/urdf/wagon.urdf (robot description, URDF)
Before this commit: robot wagon, 11 links, 10 joints
Links:
- added link rtk_pole, mass 0.314; collision cylinder length=0.28 radius=0.01; visual cylinder length=0.28 radius=0.01
Joints:
- added joint rtk_joint: type fixed, parent base_link, child rtk_pole, origin xyz=-0.200 0 0.42200000000000004 rpy=0 0 0

File: wagon_description/urdf/wagon.xacro (robot description, xacro)
@@ -229,5 +229,5 @@
     </visual>
     <collision>
-      <origin xyz="0 0 -0.036" rpy="0 0 0"/>
+      <origin xyz="0 0 0" rpy="0 0 0"/>
       <geometry>
         <cylinder length="0.072" radius="0.079"/>
@@ -240,3 +240,30 @@
     </inertial>
   </link>
+  <xacro:property name="rtk_pole_height" value="0.28" />
+  <joint name="rtk_joint" type="fixed">
+    <parent link="base_link"/>
+    <child link="rtk_pole"/>
+    <origin xyz="-0.200 0 ${0.142+rtk_pole_height}" rpy="0 0 0"/>
+  </joint>
+  <link name="rtk_pole">
+    <visual>
+      <origin xyz="0 0 -${rtk_pole_height/2}" rpy="0 0 0"/>
+      <geometry>
+        <!-- <mesh filename="package://wagon_description/meshes/sensors/rtk.dae" scale="1 1 1"/> -->
+        <cylinder length="${rtk_pole_height}" radius="0.01"/>
+      </geometry>
+      <material name="dark"/>
+    </visual>
+    <collision>
+      <origin xyz="0 0 -${rtk_pole_height/2}" rpy="0 0 0"/>
+      <geometry>
+        <cylinder length="${rtk_pole_height}" radius="0.01"/>
+      </geometry>
+    </collision>
+    <inertial>
+      <mass value="0.314" />
+      <origin xyz="0 0 0" />
+      <inertia ixx="0.001" ixy="0.0" ixz="0.0" iyy="0.001" iyz="0.0" izz="0.001" />
+    </inertial>
+  </link>
 </robot>

Commit message: fixed opposite turning of hydraulic joint

File: wagon_description/urdf/wagon.urdf (robot description, URDF)
Before this commit: robot wagon, 12 links, 11 joints
Joints:
- joint hydraulic_joint: axis 0 0 1 -> 0 0 -1; limit lower=-0.70 upper=0.70 effort=1000.0 velocity=0.5 -> lower=-0.80 upper=0.80 effort=1000.0 velocity=0.5

File: wagon_description/urdf/wagon.xacro (robot description, xacro)
@@ -44,6 +44,6 @@
     </link>
   <joint name="hydraulic_joint" type="revolute">
-    <axis xyz="0 0 1"/>
-    <limit effort="1000.0" lower="-0.70" upper="0.70" velocity="0.5"/>
+    <axis xyz="0 0 -1"/>
+    <limit effort="1000.0" lower="-0.80" upper="0.80" velocity="0.5"/>
     <origin rpy="0 0 0" xyz="0.0 0.0 0"/>
     <parent link="connection_link"/>

Commit message: Added launch file for odom and added to bringup

File: wagon_description/urdf/wagon.urdf (robot description, URDF)
Before this commit: robot wagon, 12 links, 11 joints
Links:
- removed link base_footprint
- link base_link: mass 135.5 -> 185.5
- link rear_link: mass 140.5 -> 190.5
Joints:
- removed joint base_joint
- joint imu_joint: parent base_link -> rear_link

File: wagon_description/urdf/wagon.xacro (robot description, xacro)
@@ -5,4 +5,6 @@
   <xacro:property name="hydraulic_offset" value="0.085" />
   <xacro:property name="rear_link_offset" value="-0.8716" />
+  <xacro:property name="base_link_offset" value="0.6948" />
+<!--
   <link name="base_footprint">
   </link>
@@ -11,5 +13,5 @@
     <child link="base_link"/>
     <origin xyz="0.6948 0 0" rpy="0 0 0"/>
-  </joint>
+  </joint> -->
   <link name="base_link">
     <visual>
@@ -21,5 +23,5 @@
     </visual>
     <collision>
-      <origin xyz="-${0.6948-(1.055/2)+0.02} 0 0" rpy="0 0 0"/>
+      <origin xyz="-${base_link_offset-(1.055/2)+0.02} 0 0" rpy="0 0 0"/>
       <geometry>
         <box size="1.055 0.620 0.260"/>
@@ -28,5 +30,5 @@
     <inertial>
       <origin xyz="-0.142 0 0" rpy="0 ${pi/2} 0" />
-      <mass value="135.5" />
+      <mass value="185.5" />
       <inertia ixx="6.189"
                ixy="0" iyy="17.997"
@@ -76,5 +78,5 @@
     <inertial>
         <origin xyz="${0.142} 0 0" rpy="0 0 0" />
-        <mass value="140.5" />
+        <mass value="190.5" />
       <inertia ixx="6.189"
                ixy="0" iyy="17.997"
@@ -210,5 +212,5 @@
   </link>
   <joint name="imu_joint" type="fixed">
-    <parent link="base_link"/>
+    <parent link="rear_link"/>
     <child link="imu_link"/>
     <origin xyz="-0.032 0 0.068" rpy="0 0 0"/>

Commit message: updated odom

File: wagon_description/urdf/wagon.urdf (robot description, URDF)
Before this commit: robot wagon, 11 links, 10 joints
Links:
- removed link imu_link
- added link base_scan_imu_link
- added link rear_imu_link
Joints:
- removed joint imu_joint
- added joint base_scan_imu_joint: type fixed, parent base_scan, child base_scan_imu_link, origin xyz=0.0 0.0 0.0 rpy=0 0 0
- added joint rear_imu_joint: type fixed, parent rear_link, child rear_imu_link, origin xyz=-0.032 0 0.068 rpy=0 0 0
- joint scan_joint: origin xyz=0 0 0.272 rpy=0 0 0 -> xyz=0 0 1.0 rpy=0 0 0

File: wagon_description/urdf/wagon.xacro (robot description, xacro)
@@ -211,14 +211,20 @@
     </inertial>
   </link>
-  <joint name="imu_joint" type="fixed">
+  <joint name="rear_imu_joint" type="fixed">
     <parent link="rear_link"/>
-    <child link="imu_link"/>
+    <child link="rear_imu_link"/>
     <origin xyz="-0.032 0 0.068" rpy="0 0 0"/>
   </joint>
-  <link name="imu_link"/>
+  <link name="rear_imu_link"/>
+  <joint name="base_scan_imu_joint" type="fixed">
+    <parent link="base_scan"/>
+    <child link="base_scan_imu_link"/>
+    <origin xyz="0.0 0.0 0.0" rpy="0 0 0"/>
+  </joint>
+  <link name="base_scan_imu_link"/>
   <joint name="scan_joint" type="fixed">
     <parent link="base_link"/>
     <child link="base_scan"/>
-    <origin xyz="0 0 0.272" rpy="0 0 0"/>
+    <origin xyz="0 0 1.0" rpy="0 0 0"/>
   </joint>
   <link name="base_scan">
